File: hardware/Delfino_Audio_Cape/DAC_Filter.sch (KiCad schematic (older format))
At the start: 12 parts, among them U1 TL082

Commit message: Avances de la tarjeta de expansión
Parts:
- C19: renamed from C1; footprint (none) -> Capacitors_THT:C_Disc_D4.3mm_W1.9mm_P5.00mm
- C20: renamed from C2; footprint (none) -> Capacitors_THT:CP_Radial_D6.3mm_P2.50mm
- C21: renamed from C4; footprint (none) -> Capacitors_THT:C_Disc_D4.3mm_W1.9mm_P5.00mm
- C22: renamed from C3; footprint (none) -> Capacitors_THT:C_Disc_D4.3mm_W1.9mm_P5.00mm
- C23: renamed from C5; footprint (none) -> Capacitors_THT:CP_Radial_D6.3mm_P2.50mm
- R32: renamed from R1; footprint (none) -> Resistors_THT:R_Axial_DIN0207_L6.3mm_D2.5mm_P10.16mm_Horizontal
- R33: renamed from R2; footprint (none) -> Resistors_THT:R_Axial_DIN0207_L6.3mm_D2.5mm_P10.16mm_Horizontal
- R34: renamed from R3; footprint (none) -> Resistors_THT:R_Axial_DIN0207_L6.3mm_D2.5mm_P10.16mm_Horizontal
- R35: renamed from R4; footprint (none) -> Resistors_THT:R_Axial_DIN0207_L6.3mm_D2.5mm_P10.16mm_Horizontal
- R36: renamed from R5; footprint (none) -> Resistors_THT:R_Axial_DIN0207_L6.3mm_D2.5mm_P10.16mm_Horizontal
- R37: renamed from R?; footprint (none) -> Resistors_THT:R_Axial_DIN0207_L6.3mm_D2.5mm_P10.16mm_Horizontal
- U4: renamed from U1; footprint (none) -> Housings_DIP:DIP-8_W7.62mm_LongPads
Changed lines of the file:
@@
 LIBS:contrib
 LIBS:valves
-LIBS:My_Audio_Conn
 LIBS:Delfino_Audio_Cape-cache
 EELAYER 25 0
@@
 $Descr A4 11693 8268
 encoding utf-8
-Sheet 6 6
+Sheet 4 6
 Title ""
 Date ""
@@
 $EndDescr
 $Comp
-L TL082 U1
+L TL082 U4
 U 1 1 599B6267
 P 6150 2700
-F 0 "U1" H 6150 2900 50  0000 L CNN
+AR Path="/59BA7873/599B6267" Ref="U4"  Part="1"
+AR Path="/59BA9CE1/599B6267" Ref="U4"  Part="2"
+AR Path="/59BC9EFF/599B6267" Ref="U5"  Part="1"
+F 0 "U5" H 6150 2900 50  0000 L CNN
 F 1 "TL082" H 6150 2500 50  0000 L CNN
-F 2 "" H 6150 2700 50  0001 C CNN
+F 2 "Housings_DIP:DIP-8_W7.62mm_LongPads" H 6150 2700 50  0001 C CNN
 F 3 "" H 6150 2700 50  0001 C CNN
 	1    6150 2700
@@
 $EndComp
 $Comp
-L C C1
+L C C19
 U 1 1 599B62D2
 P 3600 2600
-F 0 "C1" V 3540 2440 50  0000 L CNN
+AR Path="/59BA7873/599B62D2" Ref="C19"  Part="1"
+AR Path="/59BA9CE1/599B62D2" Ref="C24"  Part="1"
+AR Path="/59BC9EFF/599B62D2" Ref="C29"  Part="1"
+F 0 "C29" V 3540 2440 50  0000 L CNN
 F 1 "220nF" V 3540 2660 50  0000 L CNN
-F 2 "" H 3638 2450 50  0001 C CNN
+F 2 "Capacitors_THT:C_Disc_D4.3mm_W1.9mm_P5.00mm" H 3638 2450 50  0001 C CNN
 F 3 "" H 3600 2600 50  0001 C CNN
 	1    3600 2600
@@
 $EndComp
 $Comp
-L R R1
+L R R32
 U 1 1 599B6345
 P 3950 2840
-F 0 "R1" V 4030 2840 50  0000 C CNN
+AR Path="/59BA7873/599B6345" Ref="R32"  Part="1"
+AR Path="/59BA9CE1/599B6345" Ref="R38"  Part="1"
+AR Path="/59BC9EFF/599B6345" Ref="R44"  Part="1"
+F 0 "R44" V 4030 2840 50  0000 C CNN
 F 1 "1.2M" V 3950 2840 50  0000 C CNN
-F 2 "" V 3880 2840 50  0001 C CNN
+F 2 "Resistors_THT:R_Axial_DIN0207_L6.3mm_D2.5mm_P10.16mm_Horizontal" V 3880 2840 50  0001 C CNN
 F 3 "" H 3950 2840 50  0001 C CNN
 	1    3950 2840
@@
 $EndComp
 $Comp
-L R R2
+L R R33
 U 1 1 599B68B9
 P 4260 2600
-F 0 "R2" V 4340 2600 50  0000 C CNN
+AR Path="/59BA7873/599B68B9" Ref="R33"  Part="1"
+AR Path="/59BA9CE1/599B68B9" Ref="R39"  Part="1"
+AR Path="/59BC9EFF/599B68B9" Ref="R45"  Part="1"
+F 0 "R45" V 4340 2600 50  0000 C CNN
 F 1 "5.1K" V 4260 2600 50  0000 C CNN
-F 2 "" V 4190 2600 50  0001 C CNN
+F 2 "Resistors_THT:R_Axial_DIN0207_L6.3mm_D2.5mm_P10.16mm_Horizontal" V 4190 2600 50  0001 C CNN
 F 3 "" H 4260 2600 50  0001 C CNN
 	1    4260 2600
@@
 $EndComp
 $Comp
-L R R5
+L R R36
 U 1 1 599B6936
 P 4850 2600
-F 0 "R5" V 4930 2600 50  0000 C CNN
+AR Path="/59BA7873/599B6936" Ref="R36"  Part="1"
+AR Path="/59BA9CE1/599B6936" Ref="R42"  Part="1"
+AR Path="/59BC9EFF/599B6936" Ref="R48"  Part="1"
+F 0 "R48" V 4930 2600 50  0000 C CNN
 F 1 "10K" V 4850 2600 50  0000 C CNN
-F 2 "" V 4780 2600 50  0001 C CNN
+F 2 "Resistors_THT:R_Axial_DIN0207_L6.3mm_D2.5mm_P10.16mm_Horizontal" V 4780 2600 50  0001 C CNN
 F 3 "" H 4850 2600 50  0001 C CNN
 	1    4850 2600
@@
 $EndComp
 $Comp
-L C C4
+L C C21
 U 1 1 599B69B0
 P 5120 1940
-F 0 "C4" V 5070 1780 50  0000 L CNN
+AR Path="/59BA7873/599B69B0" Ref="C21"  Part="1"
+AR Path="/59BA9CE1/599B69B0" Ref="C26"  Part="1"
+AR Path="/59BC9EFF/599B69B0" Ref="C31"  Part="1"
+F 0 "C31" V 5070 1780 50  0000 L CNN
 F 1 "2.2nF" V 5070 2000 50  0000 L CNN
-F 2 "" H 5158 1790 50  0001 C CNN
+F 2 "Capacitors_THT:C_Disc_D4.3mm_W1.9mm_P5.00mm" H 5158 1790 50  0001 C CNN
 F 3 "" H 5120 1940 50  0001 C CNN
 	1    5120 1940
@@
 $EndComp
 $Comp
-L C C3
+L C C22
 U 1 1 599B6A43
 P 5180 3040
-F 0 "C3" H 5205 3140 50  0000 L CNN
+AR Path="/59BA7873/599B6A43" Ref="C22"  Part="1"
+AR Path="/59BA9CE1/599B6A43" Ref="C27"  Part="1"
+AR Path="/59BC9EFF/599B6A43" Ref="C32"  Part="1"
+F 0 "C32" H 5205 3140 50  0000 L CNN
 F 1 "1nF" H 5205 2940 50  0000 L CNN
-F 2 "" H 5218 2890 50  0001 C CNN
+F 2 "Capacitors_THT:C_Disc_D4.3mm_W1.9mm_P5.00mm" H 5218 2890 50  0001 C CNN
 F 3 "" H 5180 3040 50  0001 C CNN
 	1    5180 3040
@@
 $EndComp
 $Comp
-L +12V #PWR02
+L +12V #PWR069
 U 1 1 599B8CD8
 P 6050 2340
-F 0 "#PWR02" H 6050 2190 50  0001 C CNN
+AR Path="/59BA7873/599B8CD8" Ref="#PWR069"  Part="1"
+AR Path="/59BA9CE1/599B8CD8" Ref="#PWR075"  Part="1"
+AR Path="/59BC9EFF/599B8CD8" Ref="#PWR081"  Part="1"
+F 0 "#PWR081" H 6050 2190 50  0001 C CNN
 F 1 "+12V" H 6050 2480 50  0000 C CNN
 F 2 "" H 6050 2340 50  0001 C CNN
@@
 $EndComp
 $Comp
-L GND #PWR04
+L GND #PWR070
 U 1 1 599B928E
 P 3950 3050
-F 0 "#PWR04" H 3950 2800 50  0001 C CNN
+AR Path="/59BA7873/599B928E" Ref="#PWR070"  Part="1"
+AR Path="/59BA9CE1/599B928E" Ref="#PWR076"  Part="1"
+AR Path="/59BC9EFF/599B928E" Ref="#PWR082"  Part="1"
+F 0 "#PWR082" H 3950 2800 50  0001 C CNN
 F 1 "GND" H 3950 2900 50  0000 C CNN
 F 2 "" H 3950 3050 50  0001 C CNN
@@
 $EndComp
 $Comp
-L GND #PWR05
+L GND #PWR071
 U 1 1 599B93E2
 P 5180 3260
-F 0 "#PWR05" H 5180 3010 50  0001 C CNN
+AR Path="/59BA7873/599B93E2" Ref="#PWR071"  Part="1"
+AR Path="/59BA9CE1/599B93E2" Ref="#PWR077"  Part="1"
+AR Path="/59BC9EFF/599B93E2" Ref="#PWR083"  Part="1"
+F 0 "#PWR083" H 5180 3010 50  0001 C CNN
 F 1 "GND" H 5180 3110 50  0000 C CNN
 F 2 "" H 5180 3260 50  0001 C CNN
@@
 $EndComp
 $Comp
-L GND #PWR06
+L GND #PWR072
 U 1 1 599B9406
 P 6050 3060
-F 0 "#PWR06" H 6050 2810 50  0001 C CNN
+AR Path="/59BA7873/599B9406" Ref="#PWR072"  Part="1"
+AR Path="/59BA9CE1/599B9406" Ref="#PWR078"  Part="1"
+AR Path="/59BC9EFF/599B9406" Ref="#PWR084"  Part="1"
+F 0 "#PWR084" H 6050 2810 50  0001 C CNN
 F 1 "GND" H 6050 2910 50  0000 C CNN
 F 2 "" H 6050 3060 50  0001 C CNN
@@
 $EndComp
 $Comp
-L CP C5
+L CP C23
 U 1 1 599BC824
 P 6750 2700
-F 0 "C5" H 6775 2800 50  0000 L CNN
+AR Path="/59BA7873/599BC824" Ref="C23"  Part="1"
+AR Path="/59BA9CE1/599BC824" Ref="C28"  Part="1"
+AR Path="/59BC9EFF/599BC824" Ref="C33"  Part="1"
+F 0 "C33" H 6775 2800 50  0000 L CNN
 F 1 "10uF" H 6775 2600 50  0000 L CNN
-F 2 "" H 6788 2550 50  0001 C CNN
+F 2 "Capacitors_THT:CP_Radial_D6.3mm_P2.50mm" H 6788 2550 50  0001 C CNN
 F 3 "" H 6750 2700 50  0001 C CNN
 	1    6750 2700
@@
 $EndComp
 $Comp
-L R R3
+L R R34
 U 1 1 599BCFBB
 P 4330 3840
-F 0 "R3" V 4410 3840 50  0000 C CNN
+AR Path="/59BA7873/599BCFBB" Ref="R34"  Part="1"
+AR Path="/59BA9CE1/599BCFBB" Ref="R40"  Part="1"
+AR Path="/59BC9EFF/599BCFBB" Ref="R46"  Part="1"
+F 0 "R46" V 4410 3840 50  0000 C CNN
 F 1 "10K" V 4330 3840 50  0000 C CNN
-F 2 "" V 4260 3840 50  0001 C CNN
+F 2 "Resistors_THT:R_Axial_DIN0207_L6.3mm_D2.5mm_P10.16mm_Horizontal" V 4260 3840 50  0001 C CNN
 F 3 "" H 4330 3840 50  0001 C CNN
 	1    4330 3840
@@
 $EndComp
 $Comp
-L R R4
+L R R35
 U 1 1 599BD02E
 P 4330 4230
-F 0 "R4" V 4410 4230 50  0000 C CNN
+AR Path="/59BA7873/599BD02E" Ref="R35"  Part="1"
+AR Path="/59BA9CE1/599BD02E" Ref="R41"  Part="1"
+AR Path="/59BC9EFF/599BD02E" Ref="R47"  Part="1"
+F 0 "R47" V 4410 4230 50  0000 C CNN
 F 1 "10K" V 4330 4230 50  0000 C CNN
-F 2 "" V 4260 4230 50  0001 C CNN
+F 2 "Resistors_THT:R_Axial_DIN0207_L6.3mm_D2.5mm_P10.16mm_Horizontal" V 4260 4230 50  0001 C CNN
 F 3 "" H 4330 4230 50  0001 C CNN
 	1    4330 4230
@@
 $EndComp
 $Comp
-L CP C2
+L CP C20
 U 1 1 599BD07F
 P 4080 4260
-F 0 "C2" H 4105 4360 50  0000 L CNN
+AR Path="/59BA7873/599BD07F" Ref="C20"  Part="1"
+AR Path="/59BA9CE1/599BD07F" Ref="C25"  Part="1"
+AR Path="/59BC9EFF/599BD07F" Ref="C30"  Part="1"
+F 0 "C30" H 4105 4360 50  0000 L CNN
 F 1 "10uF" H 4105 4160 50  0000 L CNN
-F 2 "" H 4118 4110 50  0001 C CNN
+F 2 "Capacitors_THT:CP_Radial_D6.3mm_P2.50mm" H 4118 4110 50  0001 C CNN
 F 3 "" H 4080 4260 50  0001 C CNN
 	1    4080 4260
@@
 $EndComp
 $Comp
-L +12V #PWR08
+L +12V #PWR073
 U 1 1 599BD1C1
 P 4330 3550
-F 0 "#PWR08" H 4330 3400 50  0001 C CNN
+AR Path="/59BA7873/599BD1C1" Ref="#PWR073"  Part="1"
+AR Path="/59BA9CE1/599BD1C1" Ref="#PWR079"  Part="1"
+AR Path="/59BC9EFF/599BD1C1" Ref="#PWR085"  Part="1"
+F 0 "#PWR085" H 4330 3400 50  0001 C CNN
 F 1 "+12V" H 4330 3690 50  0000 C CNN
 F 2 "" H 4330 3550 50  0001 C CNN
@@
 $EndComp
 $Comp
-L GND #PWR09
+L GND #PWR074
 U 1 1 599BD1F3
 P 4220 4500
-F 0 "#PWR09" H 4220 4250 50  0001 C CNN
+AR Path="/59BA7873/599BD1F3" Ref="#PWR074"  Part="1"
+AR Path="/59BA9CE1/599BD1F3" Ref="#PWR080"  Part="1"
+AR Path="/59BC9EFF/599BD1F3" Ref="#PWR086"  Part="1"
+F 0 "#PWR086" H 4220 4250 50  0001 C CNN
 F 1 "GND" H 4220 4350 50  0000 C CNN
 F 2 "" H 4220 4500 50  0001 C CNN
@@
 Voff
 $Comp
-L R R?
+L R R37
 U 1 1 59A5DF76
 P 4880 4030
-F 0 "R?" V 4960 4030 50  0000 C CNN
+AR Path="/59BA7873/59A5DF76" Ref="R37"  Part="1"
+AR Path="/59BA9CE1/59A5DF76" Ref="R43"  Part="1"
+AR Path="/59BC9EFF/59A5DF76" Ref="R49"  Part="1"
+F 0 "R49" V 4960 4030 50  0000 C CNN
 F 1 "1M" V 4880 4030 50  0000 C CNN
-F 2 "" V 4810 4030 50  0001 C CNN
+F 2 "Resistors_THT:R_Axial_DIN0207_L6.3mm_D2.5mm_P10.16mm_Horizontal" V 4810 4030 50  0001 C CNN
 F 3 "" H 4880 4030 50  0001 C CNN
 	1    4880 4030

Commit message: Avances en el PCB
Connections:
- net Voff: now also U4.5 (+); no longer U4.3 (+)
- net at C21.1, C23.1: now also U4.6 (-), U4.7; no longer U4.1, U4.2 (-)
Changed lines of the file:
@@
 LIBS:contrib
 LIBS:valves
+LIBS:My_Audio_Conn
 LIBS:Delfino_Audio_Cape-cache
 EELAYER 25 0
@@
 $Descr A4 11693 8268
 encoding utf-8
-Sheet 4 6
+Sheet 5 6
 Title ""
 Date ""
@@
 $Comp
 L TL082 U4
-U 1 1 599B6267
+U 2 1 599B6267
 P 6150 2700
 AR Path="/59BA7873/599B6267" Ref="U4"  Part="1"
 AR Path="/59BA9CE1/599B6267" Ref="U4"  Part="2"
 AR Path="/59BC9EFF/599B6267" Ref="U5"  Part="1"
-F 0 "U5" H 6150 2900 50  0000 L CNN
+F 0 "U4" H 6150 2900 50  0000 L CNN
 F 1 "TL082" H 6150 2500 50  0000 L CNN
 F 2 "Housings_DIP:DIP-8_W7.62mm_LongPads" H 6150 2700 50  0001 C CNN
 F 3 "" H 6150 2700 50  0001 C CNN
-	1    6150 2700
+	2    6150 2700
 	1    0    0    -1
 $EndComp
@@
 AR Path="/59BA9CE1/599B62D2" Ref="C24"  Part="1"
 AR Path="/59BC9EFF/599B62D2" Ref="C29"  Part="1"
-F 0 "C29" V 3540 2440 50  0000 L CNN
+F 0 "C24" V 3540 2440 50  0000 L CNN
 F 1 "220nF" V 3540 2660 50  0000 L CNN
 F 2 "Capacitors_THT:C_Disc_D4.3mm_W1.9mm_P5.00mm" H 3638 2450 50  0001 C CNN
@@
 AR Path="/59BA9CE1/599B6345" Ref="R38"  Part="1"
 AR Path="/59BC9EFF/599B6345" Ref="R44"  Part="1"
-F 0 "R44" V 4030 2840 50  0000 C CNN
+F 0 "R38" V 4030 2840 50  0000 C CNN
 F 1 "1.2M" V 3950 2840 50  0000 C CNN
 F 2 "Resistors_THT:R_Axial_DIN0207_L6.3mm_D2.5mm_P10.16mm_Horizontal" V 3880 2840 50  0001 C CNN
@@
 AR Path="/59BA9CE1/599B68B9" Ref="R39"  Part="1"
 AR Path="/59BC9EFF/599B68B9" Ref="R45"  Part="1"
-F 0 "R45" V 4340 2600 50  0000 C CNN
+F 0 "R39" V 4340 2600 50  0000 C CNN
 F 1 "5.1K" V 4260 2600 50  0000 C CNN
 F 2 "Resistors_THT:R_Axial_DIN0207_L6.3mm_D2.5mm_P10.16mm_Horizontal" V 4190 2600 50  0001 C CNN
@@
 AR Path="/59BA9CE1/599B6936" Ref="R42"  Part="1"
 AR Path="/59BC9EFF/599B6936" Ref="R48"  Part="1"
-F 0 "R48" V 4930 2600 50  0000 C CNN
+F 0 "R42" V 4930 2600 50  0000 C CNN
 F 1 "10K" V 4850 2600 50  0000 C CNN
 F 2 "Resistors_THT:R_Axial_DIN0207_L6.3mm_D2.5mm_P10.16mm_Horizontal" V 4780 2600 50  0001 C CNN
@@
 AR Path="/59BA9CE1/599B69B0" Ref="C26"  Part="1"
 AR Path="/59BC9EFF/599B69B0" Ref="C31"  Part="1"
-F 0 "C31" V 5070 1780 50  0000 L CNN
+F 0 "C26" V 5070 1780 50  0000 L CNN
 F 1 "2.2nF" V 5070 2000 50  0000 L CNN
 F 2 "Capacitors_THT:C_Disc_D4.3mm_W1.9mm_P5.00mm" H 5158 1790 50  0001 C CNN
@@
 AR Path="/59BA9CE1/599B6A43" Ref="C27"  Part="1"
 AR Path="/59BC9EFF/599B6A43" Ref="C32"  Part="1"
-F 0 "C32" H 5205 3140 50  0000 L CNN
+F 0 "C27" H 5205 3140 50  0000 L CNN
 F 1 "1nF" H 5205 2940 50  0000 L CNN
 F 2 "Capacitors_THT:C_Disc_D4.3mm_W1.9mm_P5.00mm" H 5218 2890 50  0001 C CNN
@@
 $EndComp
 $Comp
-L +12V #PWR069
+L +12V #PWR063
 U 1 1 599B8CD8
 P 6050 2340
-AR Path="/59BA7873/599B8CD8" Ref="#PWR069"  Part="1"
-AR Path="/59BA9CE1/599B8CD8" Ref="#PWR075"  Part="1"
-AR Path="/59BC9EFF/599B8CD8" Ref="#PWR081"  Part="1"
-F 0 "#PWR081" H 6050 2190 50  0001 C CNN
+AR Path="/59BA7873/599B8CD8" Ref="#PWR063"  Part="1"
+AR Path="/59BA9CE1/599B8CD8" Ref="#PWR069"  Part="1"
+AR Path="/59BC9EFF/599B8CD8" Ref="#PWR075"  Part="1"
+F 0 "#PWR075" H 6050 2190 50  0001 C CNN
 F 1 "+12V" H 6050 2480 50  0000 C CNN
 F 2 "" H 6050 2340 50  0001 C CNN
@@
 $EndComp
 $Comp
-L GND #PWR070
+L GND #PWR064
 U 1 1 599B928E
 P 3950 3050
-AR Path="/59BA7873/599B928E" Ref="#PWR070"  Part="1"
-AR Path="/59BA9CE1/599B928E" Ref="#PWR076"  Part="1"
-AR Path="/59BC9EFF/599B928E" Ref="#PWR082"  Part="1"
-F 0 "#PWR082" H 3950 2800 50  0001 C CNN
+AR Path="/59BA7873/599B928E" Ref="#PWR064"  Part="1"
+AR Path="/59BA9CE1/599B928E" Ref="#PWR070"  Part="1"
+AR Path="/59BC9EFF/599B928E" Ref="#PWR076"  Part="1"
+F 0 "#PWR076" H 3950 2800 50  0001 C CNN
 F 1 "GND" H 3950 2900 50  0000 C CNN
 F 2 "" H 3950 3050 50  0001 C CNN
@@
 $EndComp
 $Comp
-L GND #PWR071
+L GND #PWR065
 U 1 1 599B93E2
 P 5180 3260
-AR Path="/59BA7873/599B93E2" Ref="#PWR071"  Part="1"
-AR Path="/59BA9CE1/599B93E2" Ref="#PWR077"  Part="1"
-AR Path="/59BC9EFF/599B93E2" Ref="#PWR083"  Part="1"
-F 0 "#PWR083" H 5180 3010 50  0001 C CNN
+AR Path="/59BA7873/599B93E2" Ref="#PWR065"  Part="1"
+AR Path="/59BA9CE1/599B93E2" Ref="#PWR071"  Part="1"
+AR Path="/59BC9EFF/599B93E2" Ref="#PWR077"  Part="1"
+F 0 "#PWR077" H 5180 3010 50  0001 C CNN
 F 1 "GND" H 5180 3110 50  0000 C CNN
 F 2 "" H 5180 3260 50  0001 C CNN
@@
 $EndComp
 $Comp
-L GND #PWR072
+L GND #PWR066
 U 1 1 599B9406
 P 6050 3060
-AR Path="/59BA7873/599B9406" Ref="#PWR072"  Part="1"
-AR Path="/59BA9CE1/599B9406" Ref="#PWR078"  Part="1"
-AR Path="/59BC9EFF/599B9406" Ref="#PWR084"  Part="1"
-F 0 "#PWR084" H 6050 2810 50  0001 C CNN
+AR Path="/59BA7873/599B9406" Ref="#PWR066"  Part="1"
+AR Path="/59BA9CE1/599B9406" Ref="#PWR072"  Part="1"
+AR Path="/59BC9EFF/599B9406" Ref="#PWR078"  Part="1"
+F 0 "#PWR078" H 6050 2810 50  0001 C CNN
 F 1 "GND" H 6050 2910 50  0000 C CNN
 F 2 "" H 6050 3060 50  0001 C CNN
@@
 AR Path="/59BA9CE1/599BC824" Ref="C28"  Part="1"
 AR Path="/59BC9EFF/599BC824" Ref="C33"  Part="1"
-F 0 "C33" H 6775 2800 50  0000 L CNN
+F 0 "C28" H 6775 2800 50  0000 L CNN
 F 1 "10uF" H 6775 2600 50  0000 L CNN
 F 2 "Capacitors_THT:CP_Radial_D6.3mm_P2.50mm" H 6788 2550 50  0001 C CNN
@@
 AR Path="/59BA9CE1/599BCFBB" Ref="R40"  Part="1"
 AR Path="/59BC9EFF/599BCFBB" Ref="R46"  Part="1"
-F 0 "R46" V 4410 3840 50  0000 C CNN
+F 0 "R40" V 4410 3840 50  0000 C CNN
 F 1 "10K" V 4330 3840 50  0000 C CNN
 F 2 "Resistors_THT:R_Axial_DIN0207_L6.3mm_D2.5mm_P10.16mm_Horizontal" V 4260 3840 50  0001 C CNN
@@
 AR Path="/59BA9CE1/599BD02E" Ref="R41"  Part="1"
 AR Path="/59BC9EFF/599BD02E" Ref="R47"  Part="1"
-F 0 "R47" V 4410 4230 50  0000 C CNN
+F 0 "R41" V 4410 4230 50  0000 C CNN
 F 1 "10K" V 4330 4230 50  0000 C CNN
 F 2 "Resistors_THT:R_Axial_DIN0207_L6.3mm_D2.5mm_P10.16mm_Horizontal" V 4260 4230 50  0001 C CNN
@@
 AR Path="/59BA9CE1/599BD07F" Ref="C25"  Part="1"
 AR Path="/59BC9EFF/599BD07F" Ref="C30"  Part="1"
-F 0 "C30" H 4105 4360 50  0000 L CNN
+F 0 "C25" H 4105 4360 50  0000 L CNN
 F 1 "10uF" H 4105 4160 50  0000 L CNN
 F 2 "Capacitors_THT:CP_Radial_D6.3mm_P2.50mm" H 4118 4110 50  0001 C CNN
@@
 $EndComp
 $Comp
-L +12V #PWR073
+L +12V #PWR067
 U 1 1 599BD1C1
 P 4330 3550
-AR Path="/59BA7873/599BD1C1" Ref="#PWR073"  Part="1"
-AR Path="/59BA9CE1/599BD1C1" Ref="#PWR079"  Part="1"
-AR Path="/59BC9EFF/599BD1C1" Ref="#PWR085"  Part="1"
-F 0 "#PWR085" H 4330 3400 50  0001 C CNN
+AR Path="/59BA7873/599BD1C1" Ref="#PWR067"  Part="1"
+AR Path="/59BA9CE1/599BD1C1" Ref="#PWR073"  Part="1"
+AR Path="/59BC9EFF/599BD1C1" Ref="#PWR079"  Part="1"
+F 0 "#PWR079" H 4330 3400 50  0001 C CNN
 F 1 "+12V" H 4330 3690 50  0000 C CNN
 F 2 "" H 4330 3550 50  0001 C CNN
@@
 $EndComp
 $Comp
-L GND #PWR074
+L GND #PWR068
 U 1 1 599BD1F3
 P 4220 4500
-AR Path="/59BA7873/599BD1F3" Ref="#PWR074"  Part="1"
-AR Path="/59BA9CE1/599BD1F3" Ref="#PWR080"  Part="1"
-AR Path="/59BC9EFF/599BD1F3" Ref="#PWR086"  Part="1"
-F 0 "#PWR086" H 4220 4250 50  0001 C CNN
+AR Path="/59BA7873/599BD1F3" Ref="#PWR068"  Part="1"
+AR Path="/59BA9CE1/599BD1F3" Ref="#PWR074"  Part="1"
+AR Path="/59BC9EFF/599BD1F3" Ref="#PWR080"  Part="1"
+F 0 "#PWR080" H 4220 4250 50  0001 C CNN
 F 1 "GND" H 4220 4350 50  0000 C CNN
 F 2 "" H 4220 4500 50  0001 C CNN
@@
 AR Path="/59BA9CE1/59A5DF76" Ref="R43"  Part="1"
 AR Path="/59BC9EFF/59A5DF76" Ref="R49"  Part="1"
-F 0 "R49" V 4960 4030 50  0000 C CNN
+F 0 "R43" V 4960 4030 50  0000 C CNN
 F 1 "1M" V 4880 4030 50  0000 C CNN
 F 2 "Resistors_THT:R_Axial_DIN0207_L6.3mm_D2.5mm_P10.16mm_Horizontal" V 4810 4030 50  0001 C CNN
