File: hardware/Delfino_Audio_Cape/Delfino_Audio_Cape.kicad_pcb (KiCad board)
At the start: 2 copper layers, 76 parts, among them J1 JACK_PJ324, J1-J1 Conn_02x10_Counter_Clockwise, J2 JACK_PJ324, J3 JACK_PJ324, J4 JACK_PJ324, J4-J1 Conn_02x10_Counter_Clockwise, J5-J1 Conn_02x10_Counter_Clockwise, J8-J1 Conn_02x10_Counter_Clockwise, U1 TL082, U2 TL082, U3 TL082, U4 TL082

Commit message: Avances de la tarjeta de expansión
Parts:
- removed J4-J1, J5-J1, J8-J1: Conn_02x10_Counter_Clockwise, Pin_Headers:Pin_Header_Straight_2x10_Pitch2.54mm
- added C25: 10uF, Capacitors_THT:CP_Radial_D6.3mm_P2.50mm, F.Cu at (-47.0, 141.5)
- added C26: 2.2nF, Capacitors_THT:C_Disc_D4.3mm_W1.9mm_P5.00mm, F.Cu at (-46.0, 150.3)
- added C27: 1nF, Capacitors_THT:C_Disc_D4.3mm_W1.9mm_P5.00mm, F.Cu at (-53.5, 150.3)
- added C28: 10uF, Capacitors_THT:CP_Radial_D6.3mm_P2.50mm, F.Cu at (-59.8, 148.2)
- added C29: 220nF, Capacitors_THT:C_Disc_D4.3mm_W1.9mm_P5.00mm, F.Cu at (346.1, 93.4)
- added C30: 10uF, Capacitors_THT:CP_Radial_D6.3mm_P2.50mm, F.Cu at (350.9, 78.1)
- added C31: 2.2nF, Capacitors_THT:C_Disc_D4.3mm_W1.9mm_P5.00mm, F.Cu at (349.7, 86.9)
- added C32: 1nF, Capacitors_THT:C_Disc_D4.3mm_W1.9mm_P5.00mm, F.Cu at (325.9, 95.9)
- added C33: 10uF, Capacitors_THT:CP_Radial_D6.3mm_P2.50mm, F.Cu at (339.8, 91.4)
- added J1-J2: Conn_02x10_Counter_Clockwise, Pin_Headers:Pin_Header_Straight_2x10_Pitch2.54mm, F.Cu at (126.7, 103.9)
- added J1-J3: Conn_02x10_Counter_Clockwise, Pin_Headers:Pin_Header_Straight_2x10_Pitch2.54mm, F.Cu at (169.9, 40.4)
- added J1-J4: Conn_02x10_Counter_Clockwise, Pin_Headers:Pin_Header_Straight_2x10_Pitch2.54mm, F.Cu at (169.9, 103.9)
- added J5: JACK_PJ324, My_Connectors:PJ-324, F.Cu at (97.4, 232.8)
- added J6: I2C, Pin_Headers:Pin_Header_Angled_1x04_Pitch2.54mm, F.Cu at (-2.30, 230.3)
- added J7: SPI, Pin_Headers:Pin_Header_Angled_1x05_Pitch2.54mm, F.Cu at (84.1, 228.5)
- added J8: JACK_PJ324, My_Connectors:PJ-324, F.Cu at (112.7, 232.8)
- added JP1: Jumper, Pin_Headers:Pin_Header_Straight_1x02_Pitch2.54mm, F.Cu at (154.7, 17.3)
- added R41: 10K, Resistors_THT:R_Axial_DIN0207_L6.3mm_D2.5mm_P10.16mm_Horizontal, F.Cu at (-73.7, 132.7)
- added R42: 10K, Resistors_THT:R_Axial_DIN0207_L6.3mm_D2.5mm_P10.16mm_Horizontal, F.Cu at (-73.7, 139.4)
- added R43: 1M, Resistors_THT:R_Axial_DIN0207_L6.3mm_D2.5mm_P10.16mm_Horizontal, F.Cu at (-61.0, 132.7)
- added R44: 1.2M, Resistors_THT:R_Axial_DIN0207_L6.3mm_D2.5mm_P10.16mm_Horizontal, F.Cu at (336.9, 82.6)
- added R45: 5.1K, Resistors_THT:R_Axial_DIN0207_L6.3mm_D2.5mm_P10.16mm_Horizontal, F.Cu at (336.9, 75.9)
- added R46: 10K, Resistors_THT:R_Axial_DIN0207_L6.3mm_D2.5mm_P10.16mm_Horizontal, F.Cu at (325.9, 89.3)
- added R47: 10K, Resistors_THT:R_Axial_DIN0207_L6.3mm_D2.5mm_P10.16mm_Horizontal, F.Cu at (324.2, 82.6)
- added R48: 10K, Resistors_THT:R_Axial_DIN0207_L6.3mm_D2.5mm_P10.16mm_Horizontal, F.Cu at (313.1, 90.4)
- added R49: 1M, Resistors_THT:R_Axial_DIN0207_L6.3mm_D2.5mm_P10.16mm_Horizontal, F.Cu at (324.2, 75.9)
- added SW1: SW_Push, Buttons_Switches_THT:SW_PUSH_6mm, F.Cu at (38.2, 217.2)
- added SW2: SW_Push, Buttons_Switches_THT:SW_PUSH_6mm, F.Cu at (23.0, 233.5)
- added U5: TL082, Housings_DIP:DIP-8_W7.62mm_LongPads, F.Cu at (313.6, 76.0)
- C1, C19, C24, C4: value 2.2uF -> 220nF; footprint Capacitors_THT:CP_Radial_D6.3mm_P2.50mm -> Capacitors_THT:C_Disc_D4.3mm_W1.9mm_P5.00mm
- C2, C20: value 10pF -> 10uF; footprint Capacitors_THT:C_Disc_D4.3mm_W1.9mm_P5.00mm -> Capacitors_THT:CP_Radial_D6.3mm_P2.50mm
- C21: value 2.2uF -> 2.2nF; footprint Capacitors_THT:CP_Radial_D6.3mm_P2.50mm -> Capacitors_THT:C_Disc_D4.3mm_W1.9mm_P5.00mm
- C22: value 2.2uF -> 1nF; footprint Capacitors_THT:CP_Radial_D6.3mm_P2.50mm -> Capacitors_THT:C_Disc_D4.3mm_W1.9mm_P5.00mm
- C23, C3, C6: value 2.2uF -> 10uF
- C5: value 2.2uF -> 100nF; footprint Capacitors_THT:CP_Radial_D6.3mm_P2.50mm -> Capacitors_THT:C_Disc_D4.3mm_W1.9mm_P5.00mm
- J4: value JACK_PJ324 -> PWR; footprint My_Connectors:PJ-324 -> Connectors:bornier3
- R1, R5: value 10K -> 1K
- R10: value 1.5K -> 330
- R11, R9: value 10K -> 330
- R12, R16, R2, R22, R26, R36, R6: value 68K -> 10K
- R13, R23: value 47 -> 68K
- R14, R24: value 10K -> 47
- R17, R27: value 1.5K -> 68K
- R18, R28: value 15K -> 1.5K
- R19, R29: value 10K -> 15K
- R20, R30, R40: value 1.5K -> 10K
- R21, R31: value 10K -> 1.5K
- R3: value 47 -> R
- R32: value 68K -> 1.2M
- R33: value 47 -> 5.1K
- R37: value 1.5K -> 1M
- R38: value 15K -> 1.2M
- R39: value 10K -> 5.1K
- R4: value 10K -> R
- R7: value 1.5K -> R
- R8: value 15K -> R
- U1: value TL082 -> L7812; footprint Housings_DIP:DIP-8_W7.62mm_LongPads -> TO_SOT_Packages_THT:TO-220_Horizontal
- moved C7 436.1 mm to (-142.9, -70.0), turned to 180 degrees
- moved C12 429.3 mm to (-123.9, -80.9), turned to 180 degrees
- moved C10 421.7 mm to (-117.1, -75.9)
- moved C9 421.0 mm to (-136.8, -67.5), turned to 270 degrees
- moved R13 417.8 mm to (-134.8, -75.9), turned to 180 degrees
- moved C8 408.9 mm to (-134.8, -72.8), turned to 180 degrees
- moved C11 401.0 mm to (-105.1, -63.4), turned to 270 degrees
- moved R19 396.9 mm to (-120.0, -64.2)
- moved R16 395.6 mm to (-128.7, -61.4), turned to 270 degrees
- moved R18 391.3 mm to (-120.0, -68.0)
- moved R14 387.3 mm to (-121.4, -75.9), turned to 180 degrees
- moved R12 386.8 mm to (-133.0, -51.2), turned to 90 degrees
- moved U2 385.9 mm to (-131.5, -72.6)
- moved R15 385.1 mm to (-124.1, -51.2), turned to 90 degrees
- moved R17 379.2 mm to (-100.2, -75.9), turned to 180 degrees
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Connections:
- C1 pad 1: Net-(C1-Pad1) -> /GPIO_2
- C1 pad 2: /Mic_1 -> GND
- C10 pad 2: /Mic_Amp2/Vpre -> /Mic_Amp1/Vpre
- C11 pad 2: /ADC_A1 -> /ADC_A2
- C13 pad 2: /Mic_3 -> /Mic_2
- C15 pad 1: /Mic_Amp3/Voff -> /Mic_Amp2/Voff
- C16 pad 2: /Mic_Amp3/Vpre -> /Mic_Amp2/Vpre
- C17 pad 2: /ADC_A2 -> /ADC_A3
- C19 pad 2: /Mic_4 -> /ADC_A0
- C2 pad 1: Net-(C2-Pad1) -> /Aux_L
- C2 pad 2: Net-(C1-Pad1) -> /ADC_B2
- C20 pad 2: Net-(C19-Pad1) -> GND
- C21 pad 1: /Mic_Amp4/Voff -> Net-(C21-Pad1)
- C21 pad 2: GND -> Net-(C21-Pad2)
- C22 pad 1: Net-(C22-Pad1) -> /DAC_Filter1/Voff
- C22 pad 2: /Mic_Amp4/Vpre -> GND
- C23 pad 1: Net-(C23-Pad1) -> Net-(C21-Pad1)
- C23 pad 2: /ADC_A3 -> /Out_L
- C24 pad 1: +12V -> Net-(C24-Pad1)
- C24 pad 2: GND -> /ADC_A1
- C3 pad 1: /Mic_Amp1/Voff -> Net-(C3-Pad1)
- C4 pad 1: Net-(C4-Pad1) -> /GPIO_3
- C4 pad 2: /Mic_Amp1/Vpre -> GND
- C5 pad 1: Net-(C5-Pad1) -> +12V
- C5 pad 2: /ADC_A0 -> GND
- C6 pad 1: +12V -> /Aux_R
- C6 pad 2: GND -> /ADC_B3
- C7 pad 2: /Mic_2 -> /Mic_1
- C9 pad 1: /Mic_Amp2/Voff -> /Mic_Amp1/Voff
- J1 pad 1: (no net) -> GND
- J1 pad 2: /Mic_1 -> /Aux_R
- J1 pad 3: (no net) -> /Aux_R
- J1 pad 4: (no net) -> /Aux_L
- J1 pad 5: (no net) -> /Aux_L
- J1-J1 pad 1: (no net) -> +3V3
- J1-J1 pad 10: (no net) -> /I2CA_SDA
- J1-J1 pad 12: (no net) -> /ADC_A1
- J1-J1 pad 14: (no net) -> /ADC_A0
- J1-J1 pad 15: (no net) -> /ADC_B2
- J1-J1 pad 17: (no net) -> /ADC_B1
- J1-J1 pad 19: (no net) -> GND
- J1-J1 pad 20: (no net) -> +5V
- J1-J1 pad 7: /ADC_A0 -> /SPIA_CLK
- J1-J1 pad 9: /ADC_A1 -> /I2CA_SCL
- J2 pad 1: (no net) -> GND
- J2 pad 2: /Mic_2 -> /Mic_1
- J2 pad 3: (no net) -> /Mic_1
- J2 pad 4: (no net) -> /Mic_1
- J2 pad 5: (no net) -> /Mic_1
- J3 pad 1: (no net) -> GND
- J3 pad 2: /Mic_3 -> /Mic_2
- J3 pad 3: (no net) -> /Mic_2
- J3 pad 4: (no net) -> /Mic_2
- J3 pad 5: (no net) -> /Mic_2
- J4 pad 1: (no net) -> VCC
- J4 pad 2: /Mic_4 -> (no net)
- J4 pad 3: (no net) -> GND
- R1 pad 1: +12V -> /GPIO_2
- R1 pad 2: /Mic_1 -> Net-(R1-Pad2)
- R10 pad 1: GND -> /PWM_8A
- R10 pad 2: /ADC_A0 -> (no net)
- R11 pad 1: +12V -> /PWM_6A
- R11 pad 2: /Mic_2 -> (no net)
- R12 pad 1: Net-(C8-Pad1) -> +12V
- R12 pad 2: Net-(C7-Pad1) -> /Mic_1
- R13 pad 1: Net-(C10-Pad1) -> Net-(C8-Pad1)
- R13 pad 2: Net-(C8-Pad1) -> Net-(C7-Pad1)
- R14 pad 1: +12V -> Net-(C10-Pad1)
- R14 pad 2: /Mic_Amp2/Voff -> Net-(C8-Pad1)
- R15 pad 1: /Mic_Amp2/Voff -> +12V
- R15 pad 2: GND -> /Mic_Amp1/Voff
- R16 pad 1: GND -> /Mic_Amp1/Voff
- R16 pad 2: /Mic_Amp2/Vpre -> GND
- R17 pad 1: Net-(R17-Pad1) -> GND
- R17 pad 2: /Mic_Amp2/Vpre -> /Mic_Amp1/Vpre
- R18 pad 1: Net-(R17-Pad1) -> Net-(R18-Pad1)
- R18 pad 2: Net-(C11-Pad1) -> /Mic_Amp1/Vpre
- R19 pad 1: +12V -> Net-(R18-Pad1)
- R19 pad 2: /ADC_A1 -> Net-(C11-Pad1)
- R2 pad 1: Net-(C2-Pad1) -> /GPIO_2
- R2 pad 2: Net-(C1-Pad1) -> +3V3
- R20 pad 1: GND -> +12V
- R20 pad 2: /ADC_A1 -> /ADC_A2
- R21 pad 1: +12V -> GND
- R21 pad 2: /Mic_3 -> /ADC_A2
- R22 pad 1: Net-(C14-Pad1) -> +12V
- R22 pad 2: Net-(C13-Pad1) -> /Mic_2
- R23 pad 1: Net-(C16-Pad1) -> Net-(C14-Pad1)
- R23 pad 2: Net-(C14-Pad1) -> Net-(C13-Pad1)
- R24 pad 1: +12V -> Net-(C16-Pad1)
- R24 pad 2: /Mic_Amp3/Voff -> Net-(C14-Pad1)
- R25 pad 1: /Mic_Amp3/Voff -> +12V
- R25 pad 2: GND -> /Mic_Amp2/Voff
- R26 pad 1: GND -> /Mic_Amp2/Voff
- R26 pad 2: /Mic_Amp3/Vpre -> GND
- R27 pad 1: Net-(R27-Pad1) -> GND
- R27 pad 2: /Mic_Amp3/Vpre -> /Mic_Amp2/Vpre
- R28 pad 1: Net-(R27-Pad1) -> Net-(R28-Pad1)
- R28 pad 2: Net-(C17-Pad1) -> /Mic_Amp2/Vpre
- R29 pad 1: +12V -> Net-(R28-Pad1)
- R29 pad 2: /ADC_A2 -> Net-(C17-Pad1)
- R3 pad 1: Net-(C4-Pad1) -> +12V
- R3 pad 2: Net-(C2-Pad1) -> /ADC_B2
- R30 pad 1: GND -> +12V
- R30 pad 2: /ADC_A2 -> /ADC_A3
- R31 pad 1: +12V -> GND
- R31 pad 2: /Mic_4 -> /ADC_A3
- R32 pad 1: Net-(C20-Pad1) -> Net-(C19-Pad1)
- R32 pad 2: Net-(C19-Pad1) -> GND
- R33 pad 1: Net-(C22-Pad1) -> Net-(C21-Pad2)
- R33 pad 2: Net-(C20-Pad1) -> Net-(C19-Pad1)
- R34 pad 2: /Mic_Amp4/Voff -> Net-(C20-Pad1)
- R35 pad 1: /Mic_Amp4/Voff -> Net-(C20-Pad1)
- R36 pad 1: GND -> /DAC_Filter1/Voff
- R36 pad 2: /Mic_Amp4/Vpre -> Net-(C21-Pad2)
- R37 pad 1: Net-(R37-Pad1) -> /DAC_Filter1/Voff
- R37 pad 2: /Mic_Amp4/Vpre -> Net-(C20-Pad1)
- R38 pad 1: Net-(R37-Pad1) -> Net-(C24-Pad1)
- R38 pad 2: Net-(C23-Pad1) -> GND
- R39 pad 1: +12V -> Net-(C26-Pad2)
- R39 pad 2: /ADC_A3 -> Net-(C24-Pad1)
- R4 pad 1: +12V -> /ADC_B2
- R4 pad 2: /Mic_Amp1/Voff -> GND
- R40 pad 1: GND -> +12V
- R40 pad 2: /ADC_A3 -> Net-(C25-Pad1)
- R5 pad 1: /Mic_Amp1/Voff -> /GPIO_3
- R5 pad 2: GND -> Net-(R5-Pad2)
- R6 pad 1: GND -> /GPIO_3
- R6 pad 2: /Mic_Amp1/Vpre -> +3V3
- R7 pad 1: Net-(R7-Pad1) -> +12V
- R7 pad 2: /Mic_Amp1/Vpre -> /ADC_B3
- R8 pad 1: Net-(R7-Pad1) -> /ADC_B3
- R8 pad 2: Net-(C5-Pad1) -> GND
- R9 pad 1: +12V -> /PWM_9A
- R9 pad 2: /ADC_A0 -> (no net)
- U1 pad 1: Net-(C2-Pad1) -> Net-(C3-Pad1)
- U1 pad 2: Net-(C1-Pad1) -> GND
- U1 pad 3: /Mic_Amp1/Voff -> +12V
- U2 pad 3: /Mic_Amp2/Voff -> /Mic_Amp1/Voff
- U2 pad 5: /Mic_Amp2/Voff -> /Mic_Amp1/Voff
- U2 pad 6: Net-(R17-Pad1) -> Net-(R18-Pad1)
- U3 pad 3: /Mic_Amp3/Voff -> /Mic_Amp2/Voff
- U3 pad 5: /Mic_Amp3/Voff -> /Mic_Amp2/Voff
- U3 pad 6: Net-(R27-Pad1) -> Net-(R28-Pad1)
- U4 pad 1: Net-(C20-Pad1) -> Net-(C21-Pad1)
- U4 pad 2: Net-(C19-Pad1) -> Net-(C21-Pad1)
- U4 pad 3: /Mic_Amp4/Voff -> /DAC_Filter1/Voff
- U4 pad 5: /Mic_Amp4/Voff -> /DAC_Filter2/Voff
- U4 pad 6: Net-(R37-Pad1) -> Net-(C26-Pad1)
- U4 pad 7: Net-(C23-Pad1) -> Net-(C26-Pad1)
Routing:
- net +12V: track 0.00 -> 78.4 mm, vias 0 -> 2
- net /Mic_1: track 0.00 -> 24.1 mm
- net /Mic_Amp1/Voff: track 0.00 -> 22.2 mm
- net Net-(C7-Pad1): track 0.00 -> 22.0 mm
- net Net-(C11-Pad1): track 0.00 -> 21.5 mm
- net /Mic_Amp1/Vpre: track 0.00 -> 12.3 mm
- net Net-(C8-Pad1): track 0.00 -> 10.3 mm
- net /ADC_A2: track 0.00 -> 10.2 mm
- net Net-(R18-Pad1): track 0.00 -> 7.98 mm
- net Net-(C10-Pad1): track 0.00 -> 4.32 mm
- added copper zone on B.Cu, net /Mic_1
Other:
- net class Default: trace_width 0.25 -> 0.889; via_dia 0.6 -> 2.54

Commit message: Avances en tarjeta de expansión
Parts:
- moved J3 281.5 mm to (-83.0, -50.2), turned to 90 degrees
- moved C15 68.2 mm to (-79.1, -68.0), turned to 270 degrees
- moved C13 56.3 mm to (-85.2, -70.5), turned to 180 degrees
- moved C18 49.3 mm to (-65.7, -82.2), turned to 180 degrees
- moved R30 45.7 mm to (-62.1, -56.1)
- moved C16 44.8 mm to (-58.6, -76.9)
- moved R25 40.2 mm to (-65.7, -51.7), turned to 90 degrees
- moved C17 40.0 mm to (-46.3, -64.8), turned to 270 degrees
- moved C14 39.5 mm to (-76.6, -74.1), turned to 180 degrees
- moved R23 30.5 mm to (-76.6, -76.9), turned to 180 degrees
- moved R29 29.5 mm to (-61.9, -64.8)
- moved R28 27.8 mm to (-61.9, -68.0)
- moved R26 27.2 mm to (-69.7, -61.9), turned to 270 degrees
- moved R24 22.5 mm to (-63.1, -76.9), turned to 180 degrees
- moved R27 20.5 mm to (-41.6, -76.9), turned to 180 degrees
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Routing:
- net +12V: track 78.4 -> 159.8 mm, vias 2 -> 4
- net /Mic_2: track 0.00 -> 35.5 mm
- net Net-(C13-Pad1): track 0.00 -> 23.3 mm
- net /Mic_Amp2/Voff: track 0.00 -> 22.1 mm
- net Net-(C17-Pad1): track 0.00 -> 21.8 mm
- net /Mic_Amp2/Vpre: track 0.00 -> 13.2 mm
- net /Mic_1: track 24.1 -> 36.9 mm
- net /ADC_A3: track 0.00 -> 11.0 mm
- net Net-(C14-Pad1): track 0.00 -> 9.91 mm
- net Net-(R28-Pad1): track 0.00 -> 6.98 mm
- net Net-(C16-Pad1): track 0.00 -> 4.57 mm
- added copper zone on B.Cu, net /Mic_2
Other:
- board text added: "Mic_1"
- board text added: "Mic_2"

Commit message: Avances en el PCB
Parts:
- removed J6: I2C, Pin_Headers:Pin_Header_Angled_1x04_Pitch2.54mm
- removed J7: SPI, Pin_Headers:Pin_Header_Angled_1x05_Pitch2.54mm
- added D1: LED-RGB5D-AC-R30/4P, LEDs:LED_D5.0mm-4, F.Cu at (208.6, 66.1)
- added REF**: MountingHole_2.2mm_M2_Pad, Mounting_Holes:MountingHole_2.2mm_M2_Pad, F.Cu at (250.2, 68.6)
- added REF**: MountingHole_2.2mm_M2_Pad, Mounting_Holes:MountingHole_2.2mm_M2_Pad, F.Cu at (123.2, 68.6)
- added REF**: MountingHole_2.2mm_M2_Pad, Mounting_Holes:MountingHole_2.2mm_M2_Pad, F.Cu at (250.2, 217.2)
- added REF**: MountingHole_2.2mm_M2_Pad, Mounting_Holes:MountingHole_2.2mm_M2_Pad, F.Cu at (123.2, 210.8)
- added TP1: TEST, Connectors_TestPoints:Test_Point_THTPad_4.0x4.0mm_Drill2.0mm, F.Cu at (140.6, 93.0)
- added TP10: TEST, Connectors_TestPoints:Test_Point_THTPad_4.0x4.0mm_Drill2.0mm, F.Cu at (219.8, 80.1)
- added TP11: TEST, Connectors_TestPoints:Test_Point_THTPad_4.0x4.0mm_Drill2.0mm, F.Cu at (219.8, 74.0)
- added TP12: TEST, Connectors_TestPoints:Test_Point_THTPad_4.0x4.0mm_Drill2.0mm, F.Cu at (225.3, 80.1)
- added TP13: TEST, Connectors_TestPoints:Test_Point_THTPad_4.0x4.0mm_Drill2.0mm, F.Cu at (140.6, 87.3)
- added TP14: TEST, Connectors_TestPoints:Test_Point_THTPad_4.0x4.0mm_Drill2.0mm, F.Cu at (133.6, 87.3)
- added TP15: TEST, Connectors_TestPoints:Test_Point_THTPad_4.0x4.0mm_Drill2.0mm, F.Cu at (254.1, 190.6)
- added TP16: TEST, Connectors_TestPoints:Test_Point_THTPad_4.0x4.0mm_Drill2.0mm, F.Cu at (253.3, 105.0)
- added TP17: TEST, Connectors_TestPoints:Test_Point_THTPad_4.0x4.0mm_Drill2.0mm, F.Cu at (253.3, 110.7)
- added TP18: TEST, Connectors_TestPoints:Test_Point_THTPad_4.0x4.0mm_Drill2.0mm, F.Cu at (253.3, 132.3)
- added TP19: TEST, Connectors_TestPoints:Test_Point_THTPad_4.0x4.0mm_Drill2.0mm, F.Cu at (253.3, 138.0)
- added TP2: TEST, Connectors_TestPoints:Test_Point_THTPad_4.0x4.0mm_Drill2.0mm, F.Cu at (133.6, 93.0)
- added TP20: TEST, Connectors_TestPoints:Test_Point_THTPad_4.0x4.0mm_Drill2.0mm, F.Cu at (254.1, 196.2)
- added TP3: TEST, Connectors_TestPoints:Test_Point_THTPad_4.0x4.0mm_Drill2.0mm, F.Cu at (128.3, 162.1)
- added TP4: TEST, Connectors_TestPoints:Test_Point_THTPad_4.0x4.0mm_Drill2.0mm, F.Cu at (129.5, 218.7)
- added TP5: TEST, Connectors_TestPoints:Test_Point_THTPad_4.0x4.0mm_Drill2.0mm, F.Cu at (122.4, 162.1)
- added TP6: TEST, Connectors_TestPoints:Test_Point_THTPad_4.0x4.0mm_Drill2.0mm, F.Cu at (123.4, 218.7)
- added TP7: TEST, Connectors_TestPoints:Test_Point_THTPad_4.0x4.0mm_Drill2.0mm, F.Cu at (197.6, 64.0)
- added TP8: TEST, Connectors_TestPoints:Test_Point_THTPad_4.0x4.0mm_Drill2.0mm, F.Cu at (203.2, 64.0)
- added TP9: TEST, Connectors_TestPoints:Test_Point_THTPad_4.0x4.0mm_Drill2.0mm, F.Cu at (225.3, 74.0)
- J1-J1, J1-J2, J1-J3, J1-J4: value Conn_02x10_Counter_Clockwise -> Conn_02x10_Odd_Even; footprint Pin_Headers:Pin_Header_Straight_2x10_Pitch2.54mm -> Pin_Headers:Pin_Header_Straight_2x10_Pitch2.00mm
- R3, R7: value R -> 10k
- R4, R8: value R -> 1.5k
- moved C12 348.1 mm to (148.4, 136.0), turned to 90 degrees
- moved C18 348.0 mm to (149.5, 191.3), turned to 90 degrees
- moved R27 346.3 mm to (144.1, 215.5), turned to 90 degrees
- moved R13 343.1 mm to (143.4, 125.0), turned to 90 degrees
- moved C16 341.9 mm to (144.1, 198.5), turned to 270 degrees
- moved R24 341.0 mm to (144.1, 193.9), turned to 90 degrees
- moved R14 340.7 mm to (143.4, 138.4), turned to 90 degrees
- moved C10 340.1 mm to (143.4, 142.7), turned to 270 degrees
- moved R23 339.0 mm to (144.1, 180.4), turned to 90 degrees
- moved C8 338.9 mm to (140.3, 125.0), turned to 90 degrees
- moved R17 338.8 mm to (143.4, 159.6), turned to 90 degrees
- moved U2 337.8 mm to (140.1, 128.3), turned to 270 degrees
- moved C7 337.0 mm to (137.5, 116.9), turned to 90 degrees
- moved C14 335.1 mm to (141.3, 180.4), turned to 90 degrees
- moved U3 334.0 mm to (140.3, 183.7), turned to 270 degrees
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Connections:
- C2 pad 2: /ADC_B2 -> /ADC_B4
- C6 pad 2: /ADC_B3 -> /ADC_B2
- J1-J1 pad 1: +3V3 -> (no net)
- J1-J1 pad 10: /I2CA_SDA -> /ADC_B4
- J1-J1 pad 12: /ADC_A1 -> /ADC_B2
- J1-J1 pad 15: /ADC_B2 -> (no net)
- J1-J1 pad 17: /ADC_B1 -> (no net)
- J1-J1 pad 18: (no net) -> /ADC_A1
- J1-J1 pad 19: GND -> (no net)
- J1-J1 pad 20: +5V -> (no net)
- J1-J1 pad 4: (no net) -> GND
- J1-J1 pad 7: /SPIA_CLK -> (no net)
- J1-J1 pad 8: (no net) -> /ADC_B1
- J1-J1 pad 9: /I2CA_SCL -> (no net)
- J1-J2 pad 13: /ADC_B3 -> (no net)
- J1-J2 pad 17: /ADC_A2 -> (no net)
- J1-J2 pad 19: GND -> (no net)
- J1-J2 pad 20: +5V -> (no net)
- J1-J2 pad 4: (no net) -> GND
- J1-J2 pad 8: (no net) -> /ADC_A2
- J1-J3 pad 1: (no net) -> /PWM_7A
- J1-J3 pad 14: /SPIA_SOMI -> (no net)
- J1-J3 pad 15: /SPIA_SIMO -> (no net)
- J1-J3 pad 16: /RST -> (no net)
- J1-J3 pad 2: (no net) -> GND
- J1-J3 pad 20: GND -> (no net)
- J1-J3 pad 3: /PWM_8A -> (no net)
- J1-J3 pad 5: /PWM_9A -> /PWM_8A
- J1-J3 pad 9: (no net) -> /PWM_9A
- J1-J4 pad 16: /RST -> (no net)
- J1-J4 pad 2: /GPIO_3 -> GND
- J1-J4 pad 20: GND -> (no net)
- J1-J4 pad 3: /PWM_6A -> /GPIO_3
- R10 pad 1: /PWM_8A -> /PWM_7A
- R10 pad 2: (no net) -> Net-(D1-Pad4)
- R11 pad 1: /PWM_6A -> /PWM_9A
- R11 pad 2: (no net) -> Net-(D1-Pad1)
- R3 pad 2: /ADC_B2 -> /ADC_B4
- R4 pad 1: /ADC_B2 -> /ADC_B4
- R7 pad 2: /ADC_B3 -> /ADC_B2
- R8 pad 1: /ADC_B3 -> /ADC_B2
- R9 pad 1: /PWM_9A -> /PWM_8A
- R9 pad 2: (no net) -> Net-(D1-Pad3)
Routing:
- net +12V: track 159.8 -> 729.6 mm, vias 4 -> 10
- net /ADC_B1: track 0.00 -> 105.1 mm, vias 0 -> 1
- net /ADC_A3: track 11.0 -> 98.7 mm
- net /ADC_A0: track 0.00 -> 83.0 mm
- net +3V3: track 0.00 -> 82.6 mm, vias 0 -> 2
- net /ADC_A1: track 0.00 -> 77.4 mm
- net /ADC_B2: track 0.00 -> 74.4 mm
- net /GPIO_2: track 0.00 -> 55.9 mm
- net /ADC_A2: track 10.2 -> 65.3 mm
- net /ADC_B4: track 0.00 -> 54.3 mm
- net /GPIO_3: track 0.00 -> 51.8 mm
- net /PWM_8A: track 0.00 -> 47.1 mm
- net /PWM_9A: track 0.00 -> 39.9 mm
- net /PWM_7A: track 0.00 -> 31.8 mm
- net Net-(C26-Pad1): track 0.00 -> 20.3 mm
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- added copper zone on B.Cu, net /ADC_B2
- added copper zone on B.Cu, net /ADC_B4
- added copper zone on B.Cu, net /Aux_L
- added copper zone on B.Cu, net /Aux_R
- added copper zone on B.Cu, net /Out_L
- added copper zone on B.Cu, net /Out_M
- added copper zone on B.Cu, net /Out_R
- added copper zone on F.Cu, net GND
- added copper zone on B.Cu, net Net-(C20-Pad1)
- added copper zone on B.Cu, net Net-(C25-Pad1)
- added copper zone on B.Cu, net Net-(C30-Pad1)
Other:
- board outline added: 143.8 x 162.6 mm
- net class Default: clearance 0.2 -> 0.4572
- rule trace_clearance: 0.2 -> 0.4572
- board text added: "Auxiliar"
- board text added: "Boton_1"
- board text added: "Boton_2"
- board text added: "RGB"
- board text added: "Salida_Estéreo"
- board text added: "Salida_Mono"
