File: hardware/Delfino_Audio_Cape/Delfino_Audio_Cape.sch (KiCad schematic (older format))
At the start: 20 parts, among them J1 JACK_PJ324, J1-J1 Conn_02x10_Counter_Clockwise, J1-J? Conn_02x10_Counter_Clockwise, J2 JACK_PJ324

Commit message: Avances de la tarjeta de expansión
Parts:
- removed D?: LED_RGB, symbol LED_RGB
- added C2, C3, C6: 10uF, Capacitors_THT:CP_Radial_D6.3mm_P2.50mm, symbol CP
- added C5: 100nF, Capacitors_THT:C_Disc_D4.3mm_W1.9mm_P5.00mm, symbol C
- added J1: JACK_PJ324, My_Connectors:PJ-324, symbol JACK_PJ324
- added J4: PWR, Connectors:bornier3, symbol Conn_01x03
- added J6: I2C, Pin_Headers:Pin_Header_Angled_1x04_Pitch2.54mm, symbol Conn_01x04
- added J7: SPI, Pin_Headers:Pin_Header_Angled_1x05_Pitch2.54mm, symbol Conn_01x05
- added JP1: Jumper, Pin_Headers:Pin_Header_Straight_1x02_Pitch2.54mm, symbol Jumper
- added PD1: LED-RGB5D-AC-R30/4P, Opto-Devices:KPS-5130, symbol KPS-5130
- added R3, R4, R7, R8: R, Resistors_THT:R_Axial_DIN0207_L6.3mm_D2.5mm_P10.16mm_Horizontal, symbol R
- added TP1, TP10, TP11, TP12, TP13, TP14, TP15, TP16, TP17, TP18, TP19, TP2, TP20, TP3, TP4, TP5, TP6, TP7, TP8, TP9: TEST, Measurement_Points:Measurement_Point_Square-TH_Big, symbol TEST
- added U1: L7812, TO_SOT_Packages_THT:TO-220_Horizontal, symbol L7812
- C1, C4: renamed from C?; footprint (none) -> Capacitors_THT:C_Disc_D4.3mm_W1.9mm_P5.00mm
- R1, R10, R11, R2, R5, R6, R9: renamed from R?; footprint (none) -> Resistors_THT:R_Axial_DIN0207_L6.3mm_D2.5mm_P10.16mm_Horizontal
- SW1, SW2: renamed from SW?; footprint (none) -> Buttons_Switches_THT:SW_PUSH_6mm
- gave numbers to parts that had none: 5
- renumbered J1 to J2, J2 to J3
Connections:
- net +3V3: now also J6.1 (Pin_1), J7.1 (Pin_1)
- net ADC_A2: now also TP3.1
- net ADC_A3: now also TP4.1
- net ADC_B2: now also C2.2, R3.2, R4.1, TP1.1
- net ADC_B3: now also C6.2, R7.2, R8.1, TP13.1
- net GND: now also C3.2, C5.2, J1.1 (G), J4.3 (Pin_3), J6.4 (Pin_4), J7.5 (Pin_5), PD1.4 (C), R4.2, R8.2, TP12.1, TP14.1, TP15.1, TP16.1, TP19.1, TP2.1, TP5.1, TP6.1, TP8.1, TP9.1, U1.2 (GND)
- net I2CA_SCL: now also J6.3 (Pin_3)
- net I2CA_SDA: now also J6.2 (Pin_2)
- net Out_L: now also TP17.1
- net Out_M: now also TP20.1
- net Out_R: now also TP18.1
- net PWM_8A: now also TP10.1
- net PWM_9A: now also TP11.1
- net SPIA_SIMO: now also J7.2 (Pin_2)
- net SPIA_SOMI: now also J7.3 (Pin_3)
- net at R9.2: now also PD1.3 (AB)
- net at R10.2: now also PD1.2 (AG)
- net at R11.2: now also PD1.1 (AR)
- net GPIO_60 renamed SPIA_CLK
- net SPIA_CLK: now also J7.4 (Pin_4)
- new net: C3.1, JP1.2, U1.1 (IN)
- new net +12V: C5.1, R3.1, R7.1, TP7.1, U1.3 (OUT)
- new net Aux_L: C2.1, J1.4 (LN), J1.5 (L)
- new net Aux_R: C6.1, J1.2 (R), J1.3 (RN)
- new net VCC: J4.1 (Pin_1), JP1.1
- no-connect marks 10 -> 54
Other:
- note added: "Fuente de alimentación"
- note added: "Offset para entrada auxiliar"
- moved on the sheet: J1-J1, J1-J2, J1-J3, J1-J4, J2, J3, R10, R11, R9

Commit message: Avances en el PCB
Parts:
- removed J1-J1, J1-J2, J1-J3, J1-J4: Conn_02x10_Counter_Clockwise, Pin_Headers:Pin_Header_Straight_2x10_Pitch2.54mm, symbol Conn_02x10_Counter_Clockwise
- removed J6: I2C, Pin_Headers:Pin_Header_Angled_1x04_Pitch2.54mm, symbol Conn_01x04
- removed J7: SPI, Pin_Headers:Pin_Header_Angled_1x05_Pitch2.54mm, symbol Conn_01x05
- removed PD1: LED-RGB5D-AC-R30/4P, Opto-Devices:KPS-5130, symbol KPS-5130
- added D1: LED-RGB5D-AC-R30/4P, LEDs:LED_D5.0mm-4, symbol LED_RCBG
- added J1-J1, J1-J2, J1-J3, J1-J4: Conn_02x10_Odd_Even, Pin_Headers:Pin_Header_Straight_2x10_Pitch2.00mm, symbol Conn_02x10_Odd_Even
- R3, R7: value R -> 10k
- R4, R8: value R -> 1.5k
- TP1, TP10, TP11, TP12, TP13, TP14, TP15, TP16, TP17, TP18, TP19, TP2, TP20, TP3, TP4, TP5, TP6, TP7, TP8, TP9: footprint Measurement_Points:Measurement_Point_Square-TH_Big -> Connectors_TestPoints:Test_Point_THTPad_4.0x4.0mm_Drill2.0mm
Connections:
- net +3V3: now also J1-J2.1 (Pin_1)
- net +5V: now also J1-J2.2 (Pin_2)
- net ADC_14: now also J1-J1.6 (Pin_6)
- net ADC_15: now also J1-J2.6 (Pin_6)
- net ADC_A0: now also J1-J1.14 (Pin_14)
- net ADC_A1: now also J1-J1.18 (Pin_18)
- net ADC_A2: now also J1-J2.8 (Pin_8)
- net ADC_A3: now also J1-J2.14 (Pin_14)
- net ADC_A4: now also J1-J2.18 (Pin_18)
- net ADC_A5: now also J1-J2.10 (Pin_10)
- net ADC_B0: now also J1-J1.16 (Pin_16)
- net ADC_B1: now also J1-J1.8 (Pin_8)
- net ADC_B2: now also C6.2, R7.2, R8.1, TP13.1, J1-J1.12 (Pin_12); no longer C2.2, R3.2, R4.1, TP1.1
- net ADC_B3: now also J1-J2.16 (Pin_16); no longer C6.2, R7.2, R8.1, TP13.1
- net ADC_B4: now also C2.2, R3.2, R4.1, TP1.1, J1-J1.10 (Pin_10)
- net ADC_B5: now also J1-J2.12 (Pin_12)
- net GND: now also D1.2 (K), J1-J1.4 (Pin_4), J1-J2.4 (Pin_4), J1-J3.2 (Pin_2), J1-J4.2 (Pin_2)
- net GPIO_11: now also J1-J4.7 (Pin_7)
- net GPIO_13: now also J1-J3.3 (Pin_3)
- net GPIO_15: now also J1-J3.7 (Pin_7)
- net GPIO_17: now also J1-J3.11 (Pin_11)
- net GPIO_18: now also J1-J4.9 (Pin_9)
- net GPIO_19: now also J1-J4.11 (Pin_11)
- net GPIO_2: now also J1-J4.1 (Pin_1)
- net GPIO_20: now also J1-J3.13 (Pin_13)
- net GPIO_21: now also J1-J3.15 (Pin_15)
- net GPIO_3: now also J1-J4.3 (Pin_3)
- net GPIO_4: now also J1-J3.4 (Pin_4)
- net GPIO_41: now also J1-J1.9 (Pin_9)
- net GPIO_61: now also J1-J1.15 (Pin_15)
- net GPIO_62: now also J1-J3.6 (Pin_6)
- net GPIO_63: now also J1-J4.12 (Pin_12)
- net GPIO_64: now also J1-J4.14 (Pin_14)
- net GPIO_71: now also J1-J1.3 (Pin_3)
- net GPIO_72: now also J1-J3.16 (Pin_16)
- net GPIO_73: now also J1-J3.18 (Pin_18)
- net GPIO_78: now also J1-J3.20 (Pin_20)
- net GPIO_91: now also J1-J4.4 (Pin_4)
- net GPIO_92: now also J1-J4.18 (Pin_18)
- net GPIO_99: now also J1-J4.16 (Pin_16)
- net I2CA_SCL: now also J1-J1.17 (Pin_17)
- net I2CA_SDA: now also J1-J1.19 (Pin_19)
- net I2CB_SCL: now also J1-J2.17 (Pin_17)
- net I2CB_SDA: now also J1-J2.19 (Pin_19)
- net PWM_10A: now also J1-J4.17 (Pin_17)
- net PWM_10B: now also J1-J4.19 (Pin_19)
- net PWM_11A: now also J1-J3.17 (Pin_17)
- net PWM_11B: now also J1-J3.19 (Pin_19)
- net PWM_6A: now also J1-J4.5 (Pin_5); no longer R11.1
- net PWM_8A: now also R9.1, TP11.1, J1-J3.5 (Pin_5); no longer R10.1, TP10.1
- net PWM_9A: now also R11.1, J1-J3.9 (Pin_9); no longer R9.1, TP11.1
- net SCIB_Rx: now also J1-J2.5 (Pin_5)
- net SCIB_Tx: now also J1-J2.7 (Pin_7)
- net SCIC_Rx: now also J1-J1.5 (Pin_5)
- net SCIC_Tx: now also J1-J1.7 (Pin_7)
- net SPIA_CLK: now also J1-J1.13 (Pin_13)
- net SPIA_SIMO: now also J1-J3.12 (Pin_12)
- net SPIA_SOMI: now also J1-J3.14 (Pin_14)
- net SPIB_CLK: now also J1-J2.13 (Pin_13)
- net at R9.2: now also D1.3 (BA)
- net at R10.2: now also D1.4 (GA)
- net at R11.2: now also D1.1 (RA)
- new net PWM_7A: J1-J3.1 (Pin_1), R10.1, TP10.1
- no-connect marks 54 -> 58
