File: hardware/Delfino_Audio_Cape/Delfino_Audio_Cape.sch (KiCad schematic (older format))
At the start: 52 parts, among them J1 JACK_PJ324, J1-J1 Conn_02x10_Odd_Even, J1-J2 Conn_02x10_Odd_Even, J1-J3 Conn_02x10_Odd_Even, J1-J4 Conn_02x10_Odd_Even, J2 JACK_PJ324, J3 JACK_PJ324, J4 PWR, J5 JACK_PJ324, J8 JACK_PJ324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

Commit message: Cambios en el PCB de la tarjeta de expansión
Parts:
- J1-J1, J1-J2, J1-J3, J1-J4: footprint Pin_Headers:Pin_Header_Straight_2x10_Pitch2.00mm -> Pin_Headers:Pin_Header_Straight_2x10_Pitch2.54mm
Changed lines of the file:
@@
 F 0 "J1-J1" H 5580 2350 50  0000 C CNN
 F 1 "Conn_02x10_Odd_Even" H 5580 1250 50  0000 C CNN
-F 2 "Pin_Headers:Pin_Header_Straight_2x10_Pitch2.00mm" H 5530 1850 50  0001 C CNN
+F 2 "Pin_Headers:Pin_Header_Straight_2x10_Pitch2.54mm" H 5530 1850 50  0001 C CNN
 F 3 "" H 5530 1850 50  0001 C CNN
 	1    5530 1850
@@
 F 0 "J1-J3" H 7130 2350 50  0000 C CNN
 F 1 "Conn_02x10_Odd_Even" H 7130 1250 50  0000 C CNN
-F 2 "Pin_Headers:Pin_Header_Straight_2x10_Pitch2.00mm" H 7080 1850 50  0001 C CNN
+F 2 "Pin_Headers:Pin_Header_Straight_2x10_Pitch2.54mm" H 7080 1850 50  0001 C CNN
 F 3 "" H 7080 1850 50  0001 C CNN
 	1    7080 1850
@@
 F 0 "J1-J2" H 5580 3820 50  0000 C CNN
 F 1 "Conn_02x10_Odd_Even" H 5580 2720 50  0000 C CNN
-F 2 "Pin_Headers:Pin_Header_Straight_2x10_Pitch2.00mm" H 5530 3320 50  0001 C CNN
+F 2 "Pin_Headers:Pin_Header_Straight_2x10_Pitch2.54mm" H 5530 3320 50  0001 C CNN
 F 3 "" H 5530 3320 50  0001 C CNN
 	1    5530 3320
@@
 F 0 "J1-J4" H 7130 3820 50  0000 C CNN
 F 1 "Conn_02x10_Odd_Even" H 7130 2720 50  0000 C CNN
-F 2 "Pin_Headers:Pin_Header_Straight_2x10_Pitch2.00mm" H 7080 3320 50  0001 C CNN
+F 2 "Pin_Headers:Pin_Header_Straight_2x10_Pitch2.54mm" H 7080 3320 50  0001 C CNN
 F 3 "" H 7080 3320 50  0001 C CNN
 	1    7080 3320

Commit message: Cambios en el PCB
Connections:
- net ADC_B2: now also C6.1; no longer C6.2
- net ADC_B4: now also C2.1; no longer C2.2
- net Aux_L: now also C2.2; no longer C2.1
- net Aux_R: now also C6.2; no longer C6.1
Changed lines of the file:
@@
 F 3 "" H 2070 5100 50  0001 C CNN
 	1    2070 5100
-	0    -1   -1   0
+	0    1    1    0
 $EndComp
 $Comp
@@
 F 3 "" H 3950 5100 50  0001 C CNN
 	1    3950 5100
-	0    -1   -1   0
+	0    1    1    0
 $EndComp
 $Comp
