File: hardware/Delfino_Audio_Cape/Mic_Amp.sch (KiCad schematic (older format))
At the start: 17 parts, among them U1 TL082

Commit message: Avances de la tarjeta de expansión
Parts:
- renumbered C4 to C10, C5 to C11, C6 to C12, C1 to C7, C2 to C8, C3 to C9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
