File: hardware/Delfino_Audio_Cape/Mic_Amp.sch (KiCad schematic (older format))
At the start: 17 parts, among them U2 TL082

Commit message: Cambios en el PCB
Changed lines of the file:
@@
 $Descr A4 11693 8268
 encoding utf-8
-Sheet 3 6
+Sheet 2 6
 Title "Tarjeta de expansión para el launchpad LAUNCHXL-F28377S"
 Date "2017-03-31"
@@
 AR Path="/59B9A6B7/58DB174A" Ref="U2"  Part="1"
 AR Path="/59B9DFC6/58DB174A" Ref="U3"  Part="1"
-F 0 "U3" H 4480 4300 50  0000 L CNN
+F 0 "U2" H 4480 4300 50  0000 L CNN
 F 1 "TL082" H 4480 3900 50  0000 L CNN
 F 2 "Housings_DIP:DIP-8_W7.62mm_LongPads" H 4480 4100 50  0001 C CNN
@@
 AR Path="/59B9A6B7/58DB1860" Ref="R14"  Part="1"
 AR Path="/59B9DFC6/58DB1860" Ref="R24"  Part="1"
-F 0 "R24" V 5350 4100 50  0000 C CNN
+F 0 "R14" V 5350 4100 50  0000 C CNN
 F 1 "47" V 5270 4100 50  0000 C CNN
 F 2 "Resistors_THT:R_Axial_DIN0207_L6.3mm_D2.5mm_P10.16mm_Horizontal" V 5200 4100 50  0001 C CNN
@@
 AR Path="/59B9A6B7/58DB1926" Ref="C10"  Part="1"
 AR Path="/59B9DFC6/58DB1926" Ref="C16"  Part="1"
-F 0 "C16" H 5915 4200 50  0000 L CNN
+F 0 "C10" H 5915 4200 50  0000 L CNN
 F 1 "2.2uF" H 5915 4000 50  0000 L CNN
 F 2 "Capacitors_THT:CP_Radial_D6.3mm_P2.50mm" H 5928 3950 50  0001 C CNN
@@
 AR Path="/59B9A6B7/58DB1E7D" Ref="#PWR039"  Part="1"
 AR Path="/59B9DFC6/58DB1E7D" Ref="#PWR051"  Part="1"
-F 0 "#PWR051" H 4380 4280 50  0001 C CNN
+F 0 "#PWR039" H 4380 4280 50  0001 C CNN
 F 1 "GND" H 4380 4380 50  0000 C CNN
 F 2 "" H 4380 4530 50  0001 C CNN
@@
 AR Path="/59B9A6B7/58DB209C" Ref="R15"  Part="1"
 AR Path="/59B9DFC6/58DB209C" Ref="R25"  Part="1"
-F 0 "R25" V 5640 5650 50  0000 C CNN
+F 0 "R15" V 5640 5650 50  0000 C CNN
 F 1 "10K" V 5560 5650 50  0000 C CNN
 F 2 "Resistors_THT:R_Axial_DIN0207_L6.3mm_D2.5mm_P10.16mm_Horizontal" V 5490 5650 50  0001 C CNN
@@
 AR Path="/59B9A6B7/58DB21A2" Ref="R16"  Part="1"
 AR Path="/59B9DFC6/58DB21A2" Ref="R26"  Part="1"
-F 0 "R26" V 5640 6320 50  0000 C CNN
+F 0 "R16" V 5640 6320 50  0000 C CNN
 F 1 "10K" V 5560 6320 50  0000 C CNN
 F 2 "Resistors_THT:R_Axial_DIN0207_L6.3mm_D2.5mm_P10.16mm_Horizontal" V 5490 6320 50  0001 C CNN
@@
 AR Path="/59B9A6B7/58DB2AB6" Ref="#PWR040"  Part="1"
 AR Path="/59B9DFC6/58DB2AB6" Ref="#PWR052"  Part="1"
-F 0 "#PWR052" H 5430 6270 50  0001 C CNN
+F 0 "#PWR040" H 5430 6270 50  0001 C CNN
 F 1 "GND" H 5430 6370 50  0000 C CNN
 F 2 "" H 5430 6520 50  0001 C CNN
@@
 AR Path="/59B9A6B7/58DB31C6" Ref="C7"  Part="1"
 AR Path="/59B9DFC6/58DB31C6" Ref="C13"  Part="1"
-F 0 "C13" H 3355 4300 50  0000 L CNN
+F 0 "C7" H 3355 4300 50  0000 L CNN
 F 1 "2.2uF" H 3355 4100 50  0000 L CNN
 F 2 "Capacitors_THT:CP_Radial_D6.3mm_P2.50mm" H 3368 4050 50  0001 C CNN
@@
 AR Path="/59B9A6B7/58DB599C" Ref="R12"  Part="1"
 AR Path="/59B9DFC6/58DB599C" Ref="R22"  Part="1"
-F 0 "R22" V 3020 3890 50  0000 C CNN
+F 0 "R12" V 3020 3890 50  0000 C CNN
 F 1 "10K" V 2940 3890 50  0000 C CNN
 F 2 "Resistors_THT:R_Axial_DIN0207_L6.3mm_D2.5mm_P10.16mm_Horizontal" V 2870 3890 50  0001 C CNN
@@
 AR Path="/59B9A6B7/58DB799D" Ref="R13"  Part="1"
 AR Path="/59B9DFC6/58DB799D" Ref="R23"  Part="1"
-F 0 "R23" V 4470 3260 50  0000 C CNN
+F 0 "R13" V 4470 3260 50  0000 C CNN
 F 1 "68K" V 4390 3260 50  0000 C CNN
 F 2 "Resistors_THT:R_Axial_DIN0207_L6.3mm_D2.5mm_P10.16mm_Horizontal" V 4320 3260 50  0001 C CNN
@@
 AR Path="/59B9A6B7/58DB801F" Ref="C8"  Part="1"
 AR Path="/59B9DFC6/58DB801F" Ref="C14"  Part="1"
-F 0 "C14" H 4405 3030 50  0000 L CNN
+F 0 "C8" H 4405 3030 50  0000 L CNN
 F 1 "10pF" H 4405 2830 50  0000 L CNN
 F 2 "Capacitors_THT:C_Disc_D4.3mm_W1.9mm_P5.00mm" H 4418 2780 50  0001 C CNN
@@
 AR Path="/59B9A6B7/58DB9255" Ref="R17"  Part="1"
 AR Path="/59B9DFC6/58DB9255" Ref="R27"  Part="1"
-F 0 "R27" V 6280 4300 50  0000 C CNN
+F 0 "R17" V 6280 4300 50  0000 C CNN
 F 1 "68K" V 6200 4300 50  0000 C CNN
 F 2 "Resistors_THT:R_Axial_DIN0207_L6.3mm_D2.5mm_P10.16mm_Horizontal" V 6130 4300 50  0001 C CNN
@@
 AR Path="/59B9A6B7/58DB93DB" Ref="#PWR041"  Part="1"
 AR Path="/59B9DFC6/58DB93DB" Ref="#PWR053"  Part="1"
-F 0 "#PWR053" H 6200 4260 50  0001 C CNN
+F 0 "#PWR041" H 6200 4260 50  0001 C CNN
 F 1 "GND" H 6200 4360 50  0000 C CNN
 F 2 "" H 6200 4510 50  0001 C CNN
@@
 AR Path="/59B9A6B7/58DBC635" Ref="C9"  Part="1"
 AR Path="/59B9DFC6/58DBC635" Ref="C15"  Part="1"
-F 0 "C15" H 5305 6410 50  0000 L CNN
+F 0 "C9" H 5305 6410 50  0000 L CNN
 F 1 "2.2uF" H 5305 6210 50  0000 L CNN
 F 2 "Capacitors_THT:CP_Radial_D6.3mm_P2.50mm" H 5318 6160 50  0001 C CNN
@@
 AR Path="/59B9A6B7/58DBEAEF" Ref="#PWR042"  Part="1"
 AR Path="/59B9DFC6/58DBEAEF" Ref="#PWR054"  Part="1"
-F 0 "#PWR054" H 2940 3480 50  0001 C CNN
+F 0 "#PWR042" H 2940 3480 50  0001 C CNN
 F 1 "+12V" H 2940 3770 50  0000 C CNN
 F 2 "" H 2940 3630 50  0001 C CNN
@@
 AR Path="/59B9A6B7/58DBEBDE" Ref="#PWR043"  Part="1"
 AR Path="/59B9DFC6/58DBEBDE" Ref="#PWR055"  Part="1"
-F 0 "#PWR055" H 4380 3520 50  0001 C CNN
+F 0 "#PWR043" H 4380 3520 50  0001 C CNN
 F 1 "+12V" H 4380 3810 50  0000 C CNN
 F 2 "" H 4380 3670 50  0001 C CNN
@@
 AR Path="/59B9A6B7/58DBEF77" Ref="#PWR044"  Part="1"
 AR Path="/59B9DFC6/58DBEF77" Ref="#PWR056"  Part="1"
-F 0 "#PWR056" H 5560 5290 50  0001 C CNN
+F 0 "#PWR044" H 5560 5290 50  0001 C CNN
 F 1 "+12V" H 5560 5580 50  0000 C CNN
 F 2 "" H 5560 5440 50  0001 C CNN
@@
 AR Path="/59B9A6B7/58DBFC70" Ref="#PWR045"  Part="1"
 AR Path="/59B9DFC6/58DBFC70" Ref="#PWR057"  Part="1"
-F 0 "#PWR057" H 9300 2580 50  0001 C CNN
+F 0 "#PWR045" H 9300 2580 50  0001 C CNN
 F 1 "+12V" H 9300 2870 50  0000 C CNN
 F 2 "" H 9300 2730 50  0001 C CNN
@@
 AR Path="/59B9A6B7/58DC019C" Ref="#PWR046"  Part="1"
 AR Path="/59B9DFC6/58DC019C" Ref="#PWR058"  Part="1"
-F 0 "#PWR058" H 9300 2930 50  0001 C CNN
+F 0 "#PWR046" H 9300 2930 50  0001 C CNN
 F 1 "GND" H 9300 3030 50  0000 C CNN
 F 2 "" H 9300 3180 50  0001 C CNN
@@
 AR Path="/59B9A6B7/58DC033A" Ref="C12"  Part="1"
 AR Path="/59B9DFC6/58DC033A" Ref="C18"  Part="1"
-F 0 "C18" H 9325 3060 50  0000 L CNN
+F 0 "C12" H 9325 3060 50  0000 L CNN
 F 1 "2.2uF" H 9325 2860 50  0000 L CNN
 F 2 "Capacitors_THT:CP_Radial_D6.3mm_P2.50mm" H 9338 2810 50  0001 C CNN
@@
 AR Path="/59B9A6B7/58DEB094" Ref="U2"  Part="2"
 AR Path="/59B9DFC6/58DEB094" Ref="U3"  Part="2"
-F 0 "U3" H 7400 4200 50  0000 L CNN
+F 0 "U2" H 7400 4200 50  0000 L CNN
 F 1 "TL082" H 7400 3800 50  0000 L CNN
 F 2 "Housings_DIP:DIP-8_W7.62mm_LongPads" H 7400 4000 50  0001 C CNN
@@
 AR Path="/59B9A6B7/58DED4C1" Ref="R18"  Part="1"
 AR Path="/59B9DFC6/58DED4C1" Ref="R28"  Part="1"
-F 0 "R28" V 6760 4100 50  0000 C CNN
+F 0 "R18" V 6760 4100 50  0000 C CNN
 F 1 "1.5K" V 6680 4100 50  0000 C CNN
 F 2 "Resistors_THT:R_Axial_DIN0207_L6.3mm_D2.5mm_P10.16mm_Horizontal" V 6610 4100 50  0001 C CNN
@@
 AR Path="/59B9A6B7/58DEF140" Ref="#PWR047"  Part="1"
 AR Path="/59B9DFC6/58DEF140" Ref="#PWR059"  Part="1"
-F 0 "#PWR059" H 7300 4170 50  0001 C CNN
+F 0 "#PWR047" H 7300 4170 50  0001 C CNN
 F 1 "GND" H 7300 4270 50  0000 C CNN
 F 2 "" H 7300 4420 50  0001 C CNN
@@
 AR Path="/59B9A6B7/58DEF817" Ref="#PWR048"  Part="1"
 AR Path="/59B9DFC6/58DEF817" Ref="#PWR060"  Part="1"
-F 0 "#PWR060" H 7300 3450 50  0001 C CNN
+F 0 "#PWR048" H 7300 3450 50  0001 C CNN
 F 1 "+12V" H 7300 3740 50  0000 C CNN
 F 2 "" H 7300 3600 50  0001 C CNN
@@
 AR Path="/59B9A6B7/58DF4567" Ref="R19"  Part="1"
 AR Path="/59B9DFC6/58DF4567" Ref="R29"  Part="1"
-F 0 "R29" V 7380 4850 50  0000 C CNN
+F 0 "R19" V 7380 4850 50  0000 C CNN
 F 1 "15K" V 7300 4850 50  0000 C CNN
 F 2 "Resistors_THT:R_Axial_DIN0207_L6.3mm_D2.5mm_P10.16mm_Horizontal" V 7230 4850 50  0001 C CNN
@@
 AR Path="/59B9A6B7/58DF4C3E" Ref="C11"  Part="1"
 AR Path="/59B9DFC6/58DF4C3E" Ref="C17"  Part="1"
-F 0 "C17" H 8225 4100 50  0000 L CNN
+F 0 "C11" H 8225 4100 50  0000 L CNN
 F 1 "2.2uF" H 8225 3900 50  0000 L CNN
 F 2 "Capacitors_THT:CP_Radial_D6.3mm_P2.50mm" H 8238 3850 50  0001 C CNN
@@
 AR Path="/59B9A6B7/58DF71F9" Ref="R20"  Part="1"
 AR Path="/59B9DFC6/58DF71F9" Ref="R30"  Part="1"
-F 0 "R30" V 8660 3820 50  0000 C CNN
+F 0 "R20" V 8660 3820 50  0000 C CNN
 F 1 "10K" V 8580 3820 50  0000 C CNN
 F 2 "Resistors_THT:R_Axial_DIN0207_L6.3mm_D2.5mm_P10.16mm_Horizontal" V 8510 3820 50  0001 C CNN
@@
 AR Path="/59B9A6B7/58DF7DE8" Ref="R21"  Part="1"
 AR Path="/59B9DFC6/58DF7DE8" Ref="R31"  Part="1"
-F 0 "R31" V 8660 4240 50  0000 C CNN
+F 0 "R21" V 8660 4240 50  0000 C CNN
 F 1 "1.5K" V 8580 4240 50  0000 C CNN
 F 2 "Resistors_THT:R_Axial_DIN0207_L6.3mm_D2.5mm_P10.16mm_Horizontal" V 8510 4240 50  0001 C CNN
@@
 AR Path="/59B9A6B7/58DF81C8" Ref="#PWR049"  Part="1"
 AR Path="/59B9DFC6/58DF81C8" Ref="#PWR061"  Part="1"
-F 0 "#PWR061" H 8580 4220 50  0001 C CNN
+F 0 "#PWR049" H 8580 4220 50  0001 C CNN
 F 1 "GND" H 8580 4320 50  0000 C CNN
 F 2 "" H 8580 4470 50  0001 C CNN
@@
 AR Path="/59B9A6B7/58DFAC5D" Ref="#PWR050"  Part="1"
 AR Path="/59B9DFC6/58DFAC5D" Ref="#PWR062"  Part="1"
-F 0 "#PWR062" H 8580 3440 50  0001 C CNN
+F 0 "#PWR050" H 8580 3440 50  0001 C CNN
 F 1 "+12V" H 8580 3730 50  0000 C CNN
 F 2 "" H 8580 3590 50  0001 C CNN
